Commit message: Update aron.urdf.xacro
renamed neck_link to pan_link

File: urdf/aron.urdf.xacro (robot description, xacro)
@@ -26,5 +26,5 @@
     </visual>
   </link>
-  <link name="$(arg robot_name)/neck_link">
+  <link name="$(arg robot_name)/pan_link">
     <visual>
       <origin rpy="0 0 0" xyz="0 0.0228 -0.2365"/>
@@ -40,5 +40,5 @@
     <origin rpy="0 0 0" xyz="0 -0.0228 0.2365"/>
     <parent link="$(arg robot_name)/base_link"/>
-    <child link="$(arg robot_name)/neck_link"/>
+    <child link="$(arg robot_name)/pan_link"/>
   </joint>
   <transmission name="trans_pan">
@@ -64,5 +64,5 @@
     <limit effort="3" lower="${radians(-12)}" upper="${radians(47)}" velocity="${pi}"/>
     <origin rpy="0 0 0" xyz="0 0 0.0392"/>
-    <parent link="$(arg robot_name)/neck_link"/>
+    <parent link="$(arg robot_name)/pan_link"/>
     <child link="$(arg robot_name)/tilt_link"/>
   </joint>
